Commit message: 新しいGazeboに対応

File: open_manipulator_x_description/gazebo/open_manipulator_x.gazebo.xacro (robot description, xacro)
@@ -1,7 +1,3 @@
 <?xml version="1.0"?>
-<!--
-Copied and modified from turtlebot3 example:
-https://github.com/ROBOTIS-GIT/turtlebot3/blob/kinetic-devel/turtlebot3_description/urdf/turtlebot3_waffle_pi_for_open_manipulator.gazebo.xacro
--->
 <robot xmlns:xacro="http://ros.org/wiki/xacro">
   <xacro:macro name="open_manipulator_x_gazebo" params="prefix">
@@ -26,5 +22,4 @@
       <maxVel>1.0</maxVel>
       <minDepth>0.001</minDepth>
-      <material>Gazebo/DarkGrey</material>
     </gazebo>
   </xacro:macro>
@@ -37,5 +32,4 @@
   <xacro:Link reference="${prefix}gripper_right_link"/>
   <gazebo reference="${prefix}end_effector_link">
-    <material>Gazebo/Red</material>
   </gazebo>
   <xacro:SimpleTransmission trans="${prefix}trans1" joint="${prefix}joint1" actuator="${prefix}actuator1" />

File: open_manipulator_x_description/ros2_control/open_manipulator_x_system.ros2_control.xacro (robot description, xacro)
@@ -2,8 +2,8 @@
 <robot xmlns:xacro="http://www.ros.org/wiki/xacro">
   <xacro:macro name="open_manipulator_x_system" params="name prefix port_name:=/dev/ttyUSB0 use_sim:=^|false use_fake_hardware:=^|false fake_sensor_commands:=^|false">
-    <ros2_control name="${name}" type="system">
+    <ros2_control name="omx" type="system">
       <xacro:if value="$(arg use_sim)">
         <hardware>
-          <plugin>gazebo_ros2_control/GazeboSystem</plugin>
+          <plugin>ign_ros2_control/IgnitionSystem</plugin>
         </hardware>
       </xacro:if>
@@ -21,5 +21,5 @@
             <param name="error_timeout_sec">0.2</param>
             <param name="dynamixel_model_folder">/param/dxl_model</param>
-            <param name="number_of_joints">6</param>
+            <param name="number_of_joints">5</param>
             <param name="number_of_transmissions">5</param>
             <param name="transmission_to_joint_matrix">
@@ -28,13 +28,12 @@
               0, 0, 1, 0, 0,
               0, 0, 0, 1, 0,
-              0, 0, 0, 0, 1,
-              0, 0, 0, 0, 0
+              0, 0, 0, 0, 1
             </param>
             <param name="joint_to_transmission_matrix">
-              1, 0, 0, 0, 0, 0,
-              0, 1, 0, 0, 0, 0,
-              0, 0, 1, 0, 0, 0,
-              0, 0, 0, 1, 0, 0,
-              0, 0, 0, 0, 1, 0
+              1, 0, 0, 0, 0,
+              0, 1, 0, 0, 0,
+              0, 0, 1, 0, 0,
+              0, 0, 0, 1, 0,
+              0, 0, 0, 0, 1
             </param>
             <param name="ros_update_freq">200</param>
@@ -86,12 +85,13 @@
         <state_interface name="effort"/>
       </joint>
-      <joint name="${prefix}gripper_right_joint">
-        <param name="mimic">${prefix}gripper_left_joint</param>
-        <param name="multiplier">1</param>
-        <command_interface name="position"/>
-        <state_interface name="position"/>
-        <state_interface name="velocity"/>
-        <state_interface name="effort"/>
-      </joint>
+      <xacro:if value="$(arg use_sim)">
+        <joint name="${prefix}gripper_right_joint">
+          <param name="mimic">${prefix}gripper_left_joint</param>
+          <param name="multiplier">1</param>
+          <state_interface name="position"/>
+          <state_interface name="velocity"/>
+          <state_interface name="effort"/>
+        </joint>
+      </xacro:if>
       <gpio name="dxl1">
         <param name="type">dxl</param>
@@ -106,4 +106,6 @@
         <param name="Position I Gain">100</param>
         <param name="Position D Gain">100</param>
+        <param name="Profile Velocity">200</param>
+        <param name="Profile Acceleration">50</param>
         <param name="Drive Mode">0</param>
       </gpio>
@@ -120,4 +122,6 @@
         <param name="Position I Gain">100</param>
         <param name="Position D Gain">100</param>
+        <param name="Profile Velocity">200</param>
+        <param name="Profile Acceleration">50</param>
         <param name="Drive Mode">0</param>
       </gpio>
@@ -134,4 +138,6 @@
         <param name="Position I Gain">100</param>
         <param name="Position D Gain">100</param>
+        <param name="Profile Velocity">200</param>
+        <param name="Profile Acceleration">50</param>
         <param name="Drive Mode">0</param>
       </gpio>
@@ -148,4 +154,6 @@
         <param name="Position I Gain">100</param>
         <param name="Position D Gain">100</param>
+        <param name="Profile Velocity">200</param>
+        <param name="Profile Acceleration">50</param>
         <param name="Drive Mode">0</param>
       </gpio>

File: open_manipulator_x_description/urdf/open_manipulator_x.urdf.xacro (robot description, xacro)
@@ -11,5 +11,7 @@
           <mesh filename="${meshes_file_direction}/link1.stl" scale="0.001 0.001 0.001"/>
         </geometry>
-        <material name="grey"/>
+        <material name="grey">
+          <color rgba="0.2 0.2 0.2 1"/>
+        </material>
       </visual>
       <collision>
@@ -32,5 +34,5 @@
       <origin xyz="0.012 0.0 0.017" rpy="0 0 0"/>
       <axis xyz="0 0 1"/>
-      <limit velocity="4.8" effort="1" lower="${-pi}" upper="${pi}" />
+      <limit velocity="4.8" effort="1000" lower="${-pi}" upper="${pi}" />
       <dynamics damping="0.1"/>
     </joint>
@@ -41,5 +43,7 @@
           <mesh filename="${meshes_file_direction}/link2.stl" scale="0.001 0.001 0.001"/>
         </geometry>
-        <material name="grey"/>
+        <material name="grey">
+          <color rgba="0.2 0.2 0.2 1"/>
+        </material>
       </visual>
       <collision>
@@ -62,5 +66,5 @@
       <origin xyz="0.0 0.0 0.0595" rpy="0 0 0"/>
       <axis xyz="0 1 0"/>
-      <limit velocity="4.8" effort="1" lower="${-1.5}" upper="${1.5}" />
+      <limit velocity="4.8" effort="1000" lower="${-1.5}" upper="${1.5}" />
       <dynamics damping="0.1"/>
     </joint>
@@ -71,5 +75,7 @@
           <mesh filename="${meshes_file_direction}/link3.stl" scale="0.001 0.001 0.001"/>
         </geometry>
-        <material name="grey"/>
+        <material name="grey">
+          <color rgba="0.2 0.2 0.2 1"/>
+        </material>
       </visual>
       <collision>
@@ -92,5 +98,5 @@
       <origin xyz="0.024 0 0.128" rpy="0 0 0"/>
       <axis xyz="0 1 0"/>
-      <limit velocity="4.8" effort="1" lower="${-1.5}" upper="${1.4}" />
+      <limit velocity="4.8" effort="1000" lower="${-1.5}" upper="${1.4}" />
       <dynamics damping="0.1"/>
     </joint>
@@ -101,5 +107,7 @@
           <mesh filename="${meshes_file_direction}/link4.stl" scale="0.001 0.001 0.001"/>
         </geometry>
-        <material name="grey"/>
+        <material name="grey">
+          <color rgba="0.2 0.2 0.2 1"/>
+        </material>
       </visual>
       <collision>
@@ -122,5 +130,5 @@
       <origin xyz="0.124 0.0 0.0" rpy="0 0 0"/>
       <axis xyz="0 1 0"/>
-      <limit velocity="4.8" effort="1" lower="${-1.7}" upper="${1.97}" />
+      <limit velocity="4.8" effort="1000" lower="${-1.7}" upper="${1.97}" />
       <dynamics damping="0.1"/>
     </joint>
@@ -131,5 +139,7 @@
           <mesh filename="${meshes_file_direction}/link5.stl" scale="0.001 0.001 0.001"/>
         </geometry>
-        <material name="grey"/>
+        <material name="grey">
+          <color rgba="0.2 0.2 0.2 1"/>
+        </material>
       </visual>
       <collision>
@@ -152,5 +162,5 @@
       <origin xyz="0.0817 0.021 0.0" rpy="0 0 0"/>
       <axis xyz="0 1 0"/>
-      <limit velocity="4.8" effort="1" lower="-0.010" upper="0.019" />
+      <limit velocity="4.8" effort="1000" lower="-0.010" upper="0.019" />
       <dynamics damping="0.1"/>
     </joint>
@@ -161,5 +171,7 @@
           <mesh filename="${meshes_file_direction}/gripper_left_palm.stl" scale="0.001 0.001 0.001"/>
         </geometry>
-        <material name="grey"/>
+        <material name="grey">
+          <color rgba="0.2 0.2 0.2 1"/>
+        </material>
       </visual>
       <collision>
@@ -187,7 +199,7 @@
       <origin xyz="0.0817 -0.021 0" rpy="0 0 0"/>
       <axis xyz="0 -1 0"/>
-      <limit velocity="4.8" effort="1" lower="-0.010" upper="0.019" />
+      <limit velocity="4.8" effort="1000" lower="-0.010" upper="0.019" />
+      <dynamics damping="0.7"/>
       <mimic joint="${prefix}gripper_left_joint" multiplier="1"/>
-      <dynamics damping="0.1"/>
     </joint>
     <link name="${prefix}gripper_right_link">
@@ -197,5 +209,7 @@
           <mesh filename="${meshes_file_direction}/gripper_right_palm.stl" scale="0.001 0.001 0.001"/>
         </geometry>
-        <material name="grey"/>
+        <material name="grey">
+          <color rgba="0.2 0.2 0.2 1"/>
+        </material>
       </visual>
       <collision>
@@ -224,6 +238,8 @@
           <box size="0.01 0.01 0.01" />
         </geometry>
-        <material name="red"/>
-       </visual>
+        <material name="red">
+          <color rgba="1.0 0.0 0.0 1"/>
+        </material>
+      </visual>
     </link>
   </xacro:macro>

File: open_manipulator_x_description/urdf/open_manipulator_x_robot.urdf.xacro (robot description, xacro)
@@ -7,6 +7,4 @@
   <xacro:arg name="fake_sensor_commands" default="false" />
   <xacro:arg name="port_name" default="/dev/ttyUSB0" />
-  <!-- Import Rviz colors -->
-  <xacro:include filename="$(find open_manipulator_x_description)/gazebo/materials.xacro" />
   <!-- Import all Gazebo-customization elements, including Gazebo colors -->
   <xacro:include filename="$(find open_manipulator_x_description)/gazebo/open_manipulator_x.gazebo.xacro" />
@@ -22,5 +20,5 @@
     port_name="$(arg port_name)"/>
   <gazebo>
-    <plugin name="gazebo_ros2_control" filename="libgazebo_ros2_control.so">
+    <plugin filename="libign_ros2_control-system.so" name="ign_ros2_control::IgnitionROS2ControlPlugin">
       <parameters>$(find open_manipulator_x_bringup)/config/gazebo_controller_manager.yaml</parameters>
     </plugin>
